File: inf-pkg-board.kicad_pcb (KiCad board)
At the start: 4 copper layers, 68.6 x 53.3 mm, 86 parts, among them J1 stemmaQT, J10 stemma, J4 SWD, J5 USB_C_Receptacle_USB2.0_14P, J6 ePaper Hat, J7 Conn_01x01_Pin, J8 Conn_01x01_Pin, J9 Conn_ARM_SWD_TagConnect_TC2030, Q1 AO3400A, Q2 AO3400A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

Commit message: check
Parts:
- removed Q1, Q2: AO3400A, Package_TO_SOT_SMD:SOT-23
- removed R18: 0, Resistor_SMD:R_1206_3216Metric_Pad1.30x1.75mm_HandSolder
- added C25: 100n, Capacitor_SMD:C_0402_1005Metric, F.Cu at (121.3, 79.5)
- added C26: 100n, Capacitor_SMD:C_0402_1005Metric, F.Cu at (126.2, 114.0)
- added C27: C, Capacitor_THT:C_Disc_D16.0mm_W5.0mm_P10.00mm, F.Cu at (90.1, 114.4)
- added TP_SCAP1: TestPoint, TestPoint:TestPoint_Pad_D2.5mm, F.Cu at (120.5, 108.5)
- added TP_V33_2: 3.3V_TEST, TestPoint:TestPoint_Pad_D2.0mm, F.Cu at (91.4, 77.0)
- added U1: 74LVC1G07, Package_TO_SOT_SMD:SOT-353_SC-70-5, F.Cu at (126.2, 112.0)
- added U8: 74LVC1G07, Package_TO_SOT_SMD:SOT-353_SC-70-5, F.Cu at (123.2, 82.2)
- G***: moved to B.Cu
- J7, J8, LPI1: footprint Connector_PinHeader_1.00mm:PinHeader_1x01_P1.00mm_Vertical -> Connector_PinHeader_2.54mm:PinHeader_1x01_P2.54mm_Vertical
- JP4: footprint Jumper:SolderJumper-2_P1.3mm_Bridged_Pad1.0x1.5mm -> Jumper:SolderJumper-2_P1.3mm_Open_TrianglePad1.0x1.5mm
- R12, R7: value 1M -> 100k
- moved G*** 43.3 mm to (136.3, 112.0), turned to 90 degrees
- moved C20 31.9 mm to (96.5, 118.0), turned to 180 degrees
- moved FMI1 3.31 mm to (85.5, 107.8)
- moved L1 3.28 mm to (88.4, 100.4), turned to 90 degrees
- moved R7 1.14 mm to (120.0, 81.4), turned to -90 degrees
- moved LPI1 1.07 mm to (84.2, 102.3)
- moved J7 0.85 mm to (82.0, 112.8)
- moved TP_CC_LATCH1 0.45 mm to (116.7, 79.8)
- moved JP3 0.41 mm to (137.2, 73.2)
Connections:
- net Net-(Q1-G) renamed CC_LATCH
- net Net-(Q2-S) renamed CLK_INT
- C20 pad 2: Net-(C20-Pad2) -> S_CAP
- R12 pad 1: Net-(Q2-G) -> S_CAP
- R7 pad 1: GND -> +3V3
- U4 pad 6: Net-(Q2-G) -> S_CAP
Routing:
- net S_CAP: track 0.00 -> 45.7 mm
- net Net-(Q2-G): track 23.9 -> 0.00 mm
- net +3V3: track 97.3 -> 104.4 mm, vias 18 -> 20
- net Net-(C20-Pad2): track 6.44 -> 0.00 mm
- net CLK_INT: track 23.0 -> 28.1 mm
- net Net-(LPI1-Pin_1): track 4.89 -> 8.78 mm
- net /CC_GND: track 63.7 -> 61.1 mm
- net CC_LATCH: track 31.9 -> 34.4 mm
- net GND: track 119.5 -> 117.3 mm, vias 39 -> 41
- net Net-(FMI1-Pin_1): track 2.06 -> 3.76 mm, vias 0 -> 1
- net Net-(L1-Pad2): track 1.48 -> 2.65 mm
Other:
- board text added: "2026.05"
- board text added: "3v3"
- board text added: "neither snow nor rain"
- board text added: "rev3"
- board text removed: "2026.03"
- board text removed: "return to sender"
- board text removed: "rev2"

Commit message: fixes
Other:
- board text added: "neither rain nor snow"
- board text removed: "neither snow nor rain"
Changed lines of the file:
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@@
 		)
 	)
-	(gr_text "neither snow nor rain"
+	(gr_text "neither rain nor snow"
 		(at 130 120.4 270)
 		(layer "B.SilkS")
